File: pcb/fetap.kicad_pcb (KiCad board)
At the start: 2 copper layers, 132 x 72.5 mm, 12 parts, among them SW1 SW_Push, U2 L293D, U3 Speaker Microphone, U4 stepup

Commit message: wip
Parts:
- removed Arduino Nano: Arduino_Nano_v3.x, Module:Arduino_Nano
- removed TP4056 Battery Charger: charger, suat:charger
- added A1: Arduino_Pro, Module:Arduino_Nano, F.Cu at (181.5, 33.0)
- added Charger1: charger, suat:charger, F.Cu at (64.0, 92.5)
- Hook1: renamed from Hook; value Hook -> hook switch
- Power1: renamed from Power; value Power -> VIN
- U3: value Speaker Microphone -> hoerer
- moved SW1 17.0 mm to (157.5, 87.5)
- moved StepUpModule1 3.00 mm to (44.0, 106.5)
- renumbered Battery to Battery1, Bell to J1, U4 to StepUpModule1, sim800l to sim800l1
Connections:
- Hook1 pad 2: GND -> Net-(Hook1-Pad2)
- U2 pad 1: +5V -> Net-(U2-Pad1)
Routing:
- net GND: track 368.4 -> 0.00 mm
- net +5V: track 207.3 -> 12.9 mm
- net Net-(A1-Pad25): track 114.3 -> 0.00 mm
- net Net-(A1-Pad26): track 93.9 -> 0.00 mm
- net Net-(A1-Pad23): track 60.6 -> 0.00 mm
- net Net-(A1-Pad24): track 54.3 -> 0.00 mm
- net Net-(A1-Pad6): track 41.9 -> 0.00 mm
- net Net-(U3-Pad4): track 40.0 -> 0.00 mm
- net Net-(A1-Pad7): track 39.7 -> 0.00 mm
- net Net-(U3-Pad3): track 33.9 -> 0.00 mm
- net Net-(A1-Pad12): track 28.4 -> 0.00 mm
- net Net-(U3-Pad2): track 27.9 -> 0.00 mm
- net Net-(A1-Pad10): track 26.3 -> 0.00 mm
- net Net-(sim800l1-Pad5): track 25.9 -> 0.00 mm
- net Net-(SW1-Pad2): track 25.7 -> 0.00 mm
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